Commit message: [urdf] Add root_joint in syabot
  This makes possible to fix the robot at a different place than the origin
  of the world.

File: urdf/syabot.urdf (robot description, URDF)
Before this commit: robot staubli_tx2_90, 11 links, 10 joints
Links:
- added link root
Joints:
- added joint root_joint: type fixed, parent root, child base_link, origin xyz=0.0 0.0 0.0 rpy=0.0 0.0 0.0
